File: MCU.kicad_sch (KiCad schematic)
At the start: 19 parts, among them U1 113991054, U2 SN74LVC2G17DBVR

Commit message: generated backup schematic pdfs
Other:
- title: (none) -> EauRouge
Changed lines of the file:
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@@
 	(generator_version "8.0")
 	(paper "A4")
+	(title_block
+		(title "EauRouge")
+		(date "2025-01-29")
+		(rev "1")
+	)
 	(junction
 		(at 217.17 49.53)
