File: Power.kicad_sch (KiCad schematic)
At the start: 31 parts, among them Q1 DMN3731U-7, U3 LMR51420YDDCR, U4 LM317MDCYR

Commit message: generated backup schematic pdfs
Other:
- title: (none) -> EauRouge
Changed lines of the file:
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@@
 	(generator_version "8.0")
 	(paper "A4")
+	(title_block
+		(title "EauRouge")
+		(date "2025-01-29")
+		(rev "1")
+	)
 	(junction
 		(at 186.69 147.32)
