File: EauRouge.kicad_sch (KiCad schematic)
At the start: 9 parts, among them J1 XT30PW-M, J2 SM05B-GHS-TB, J3 1985807, J4 PH1RA-03-UA, J5 PH1RA-03-UA

Commit message: generated backup schematic pdfs
Other:
- title: (none) -> EauRouge
Changed lines of the file:
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@@
 	(generator_version "8.0")
 	(paper "A4")
+	(title_block
+		(title "EauRouge")
+		(date "2025-01-29")
+		(rev "1")
+	)
 	(junction
 		(at 137.16 60.96)

Commit message: starting PCB rev 2 with perf board prototype
Parts:
- removed H1, H2, H3, H4: MountingHole, MountingHole:MountingHole_3.2mm_M3, symbol Mechanical:MountingHole
- removed J1: XT30PW-M, Connector_AMASS:AMASS_XT30PW-M_1x02_P2.50mm_Horizontal, symbol Connector:XT30PW-M
- removed J2: SM05B-GHS-TB, Connector_JST:JST_GH_SM05B-GHS-TB_1x05-1MP_P1.25mm_Horizontal, symbol Connector:JST-GH_SM05B-GHS-TB
- removed J3: 1985807, TerminalBlock_Phoenix:TerminalBlock_Phoenix_MKDS-1,5-2_1x02_P3.50mm_Horizontal_1985807, symbol Connector:Screw_Terminal_01x02_1985807
- removed J4, J5: PH1RA-03-UA, Connector_PinHeader_2.54mm:PinHeader_1x03_P2.54mm_Horizontal, symbol Connector:Conn-1x03-2.54mm-RA_PH1RA-03-UA
Other:
- removed sheet MCU
- removed sheet Power
- removed sheet Solenoid Driver
- title: EauRouge -> (none)

Commit message: fydp board rev2 starting component placement
Parts:
- added H1, H2, H3, H4: MountingHole, MountingHole:MountingHole_3.2mm_M3, symbol Mechanical:MountingHole
- added J1: SM04B-GHS-TB, Connector_JST:JST_GH_SM04B-GHS-TB_1x04-1MP_P1.25mm_Horizontal, symbol Connector:JST_GH_SM04B-GHS-TB
- added J2: XT30PW-M, Connector_AMASS:AMASS_XT30PW-M_1x02_P2.50mm_Horizontal, symbol Connector:XT30PW-M
- added J3: XT30PW-F, Connector_AMASS:AMASS_XT30PW-F_1x02_P2.50mm_Horizontal, symbol Connector:XT30PW-F
Connections:
- new net +12V: J3.2 (+)
- new net +BATT: J2.2 (+)
- new net -BATT: J2.1 (-)
- new net ESP32-RX: J1.3
- new net ESP32-TX: J1.2
- new net GND: J1.4, J1.MP
- new net SOLENOID-: J3.1 (-)
- new net USB_5V: J1.1
Other:
- added sheet 12V3A-BUCK (Buck.kicad_sch)
- added sheet Solenoid Driver (SolenoidDriver.kicad_sch)
- added sheet XIAO ESP32C3 (mcu.kicad_sch)
